File: hardware/proteus/generated/civic-workbench-rev-b.sch (EAGLE design)
At the start: 15 parts, among them J1 NodeMCU-32S, J2 3-pin CAN bench connector, J3 2-pin +5V bench supply input, U1 TJA1051T

Commit message: fix: final completion audit - bus-off disarm, TX global abort, identity, storage version
- Firmware: RX pump polls controller state while armed; bus-off or error-passive
  now disarms TX (twai_receive does not report bus-off). Mock follows the
  documented ESP-IDF return codes; regression test added.
- Host: TxScheduler.abort_all, POST /api/v1/tx/abort, UI abort button, pending
  virtual TX aborted and audited when capture stops; partial status recorded.
- Hardware identity: U1 is "NXP TJA1051 (marking 25 06 ND312)"; TJA1051T suffix
  and pin-5 variant no longer inferred; pin-5 confirmation added as open item.
- Storage: SQLite PRAGMA user_version stamped; newer layouts refused.
- UI: keyboard-operable frame rows; static accessibility tests.
- docs/reports/FINAL-COMPLETION-AUDIT.md, traceability, progress, limitations.

Co-Authored-By: Claude Opus 5.5 <noreply@anthropic.com>
Claude-Session: https://claude.ai/code/session_014trbsXF8R4Emma9DWHiz1c
Parts:
- U1: value TJA1051T -> NXP TJA1051 (marking 25 06 ND312)
Other:
- note added: "Civic-Workbench Rev B - NodeMCU-32S + NXP TJA1051 receive-only CAN"
- note removed: "Civic-Workbench Rev B - NodeMCU-32S + NXP TJA1051T receive-only CAN"
Changed lines of the file:
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@@
       <parts>
         <part name="J1" library="civic_workbench" deviceset="NODEMCU32S" device="" value="NodeMCU-32S" />
-        <part name="U1" library="civic_workbench" deviceset="TJA1051" device="" value="TJA1051T" />
+        <part name="U1" library="civic_workbench" deviceset="TJA1051" device="" value="NXP TJA1051 (marking 25 06 ND312)" />
         <part name="R1" library="civic_workbench" deviceset="R" device="" value="10k" />
         <part name="R2" library="civic_workbench" deviceset="R" device="" value="10k" />
@@
         <sheet>
           <plain>
-            <text x="25.4" y="152.4" size="3.81" layer="97">Civic-Workbench Rev B - NodeMCU-32S + NXP TJA1051T receive-only CAN</text>
+            <text x="25.4" y="152.4" size="3.81" layer="97">Civic-Workbench Rev B - NodeMCU-32S + NXP TJA1051 receive-only CAN</text>
             <text x="25.4" y="144.78" size="1.778" layer="97">U1 S pulled to +5V_CAN (Silent). GPIO21 not wired: Rev B cannot transmit.</text>
             <text x="25.4" y="139.7" size="1.778" layer="97">RXD -&gt; R3/R4 divider -&gt; GPIO22 (&lt;= 3.44 V). U1 pin 5 open (fail-safe).</text>
